File: TwinklePad.kicad_sch (KiCad schematic)
At the start: 59 parts, among them J1 Conn_01x04_Pin, J2 Conn_01x02, J4 PRT-12639, Q1 S8050, SW1 SW_Push, SW10 SW_Push, SW11 SW_Push, SW12 SW_Push, SW13 SW_Push, SW14 SW_Push, SW15 SW_Push, SW16 SW_Push, SW2 SW_Push, SW3 SW_Push, SW4 SW_Push, SW5 SW_Push, SW6 SW_Push, SW7 SW_Push, SW8 SW_Push, SW9 SW_Push

Commit message: Finished pcb, schematic and positioning - more or less
Parts:
- removed J2: Conn_01x02, Connector_PinHeader_2.54mm:PinHeader_1x02_P2.54mm_Vertical, symbol Connector_Generic:Conn_01x02
- added TP1, TP2: TestPoint, TestPoint:TestPoint_Plated_Hole_D2.0mm, symbol Connector:TestPoint
- Q1: footprint Package_TO_SOT_THT:TO-92_Inline -> Package_TO_SOT_THT:TO-92_Inline_Horizontal1
Connections:
- net VCC: now also TP1.1
- net at Q1.3 (C): now also TP2.1
Other:
- moved on the sheet: Q1
Changed lines of the file:
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@@
 	(global_label "Buzzer+"
 		(shape input)
-		(at 124.46 24.13 180)
+		(at 121.92 26.67 180)
 		(fields_autoplaced yes)
 		(effects
@@
 		)
 		(property "Intersheetrefs" "${INTERSHEET_REFS}"
-			(at 113.5524 24.13 0)
+			(at 111.0124 26.67 0)
 			(effects
 				(font
@@
 	)
 	(symbol
+		(lib_id "Connector:TestPoint")
+		(at 129.54 16.51 270)
+		(unit 1)
+		(exclude_from_sim no)
+		(in_bom yes)
+		(on_board yes)
+		(dnp no)
+		(fields_autoplaced yes)
+		(property "Reference" "TP1"
+			(at 134.62 15.2399 90)
+			(effects
+				(font
+					(size 1.27 1.27)
+				)
+				(justify left)
+			)
+		)
+		(property "Value" "TestPoint"
+			(at 134.62 17.7799 90)
+			(effects
+				(font
+					(size 1.27 1.27)
+				)
+				(justify left)
+			)
+		)
+		(property "Footprint" "TestPoint:TestPoint_Plated_Hole_D2.0mm"
+			(at 129.54 21.59 0)
+			(effects
+				(font
+					(size 1.27 1.27)
+				)
+				(hide yes)
+			)
+		)
+		(property "Datasheet" "~"
+			(at 129.54 21.59 0)
+			(effects
+				(font
+					(size 1.27 1.27)
+				)
+				(hide yes)
+			)
+		)
+		(property "Description" "test point"
+			(at 129.54 16.51 0)
+			(effects
+				(font
+					(size 1.27 1.27)
+				)
+				(hide yes)
+			)
+		)
+		(pin "1"
+		)
+		(instances
+			(project ""
+				(path "/16706bee-9459-4bee-94a4-70f692e45dc3"
+					(reference "TP1")
+					(unit 1)
+				)
+			)
+		)
+	)
+	(symbol
 		(lib_id "SK6812MINI-E:SK6812MINI-E")
 		(at 38.1 83.82 0)
@@
 	(symbol
 		(lib_id "Transistor_BJT:S8050")
-		(at 129.54 24.13 0)
+		(at 127 26.67 0)
 		(unit 1)
 		(exclude_from_sim no)
@@
 		(fields_autoplaced yes)
 		(property "Reference" "Q1"
-			(at 135.89 24.13 90)
+			(at 133.35 26.67 90)
 			(effects
 				(font
@@
 		)
 		(property "Value" "S8050"
-			(at 138.43 24.13 90)
+			(at 135.89 26.67 90)
 			(effects
 				(font
@@
 			)
 		)
-		(property "Footprint" "Package_TO_SOT_THT:TO-92_Inline"
-			(at 134.62 26.035 0)
+		(property "Footprint" "Package_TO_SOT_THT:TO-92_Inline_Horizontal1"
+			(at 132.08 28.575 0)
 			(effects
 				(font
@@
 		)
 		(property "Datasheet" "http://www.unisonic.com.tw/datasheet/S8050.pdf"
-			(at 129.54 24.13 0)
+			(at 127 26.67 0)
 			(effects
 				(font
@@
 		)
 		(property "Description" "0.7A Ic, 20V Vce, Low Voltage High Current NPN Transistor, TO-92"
-			(at 129.54 24.13 0)
+			(at 127 26.67 0)
 			(effects
 				(font
@@
 		)
 		(property "Sim.Device" "NPN"
-			(at 129.54 24.13 0)
+			(at 127 26.67 0)
 			(effects
 				(font
@@
 		)
 		(property "Sim.Pins" "1=E 2=B 3=C"
-			(at 129.54 24.13 0)
+			(at 127 26.67 0)
 			(effects
 				(font
@@
 	)
 	(symbol
-		(lib_id "Connector_Generic:Conn_01x02")
-		(at 137.16 16.51 0)
-		(unit 1)
-		(exclude_from_sim no)
-		(in_bom yes)
-		(on_board yes)
-		(dnp no)
-		(fields_autoplaced yes)
-		(property "Reference" "J2"
-			(at 139.7 16.5099 0)
-			(effects
-				(font
-					(size 1.27 1.27)
-				)
-				(justify left)
-			)
-		)
-		(property "Value" "Conn_01x02"
-			(at 139.7 19.0499 0)
-			(effects
-				(font
-					(size 1.27 1.27)
-				)
-				(justify left)
-			)
-		)
-		(property "Footprint" "Connector_PinHeader_2.54mm:PinHeader_1x02_P2.54mm_Vertical"
-			(at 137.16 16.51 0)
-			(effects
-				(font
-					(size 1.27 1.27)
-				)
-				(hide yes)
-			)
-		)
-		(property "Datasheet" "~"
-			(at 137.16 16.51 0)
-			(effects
-				(font
-					(size 1.27 1.27)
-				)
-				(hide yes)
-			)
-		)
-		(property "Description" "Generic connector, single row, 01x02, script generated (kicad-library-utils/schlib/autogen/connector/)"
-			(at 137.16 16.51 0)
-			(effects
-				(font
-					(size 1.27 1.27)
-				)
-				(hide yes)
-			)
-		)
-		(pin "1"
-		)
-		(pin "2"
-		)
-		(instances
-			(project ""
-				(path "/16706bee-9459-4bee-94a4-70f692e45dc3"
-					(reference "J2")
-					(unit 1)
-				)
-			)
-		)
-	)
-	(symbol
 		(lib_id "SK6812MINI-E:SK6812MINI-E")
 		(at 55.88 106.68 0)
@@
 	)
 	(symbol
+		(lib_id "Connector:TestPoint")
+		(at 129.54 21.59 270)
+		(unit 1)
+		(exclude_from_sim no)
+		(in_bom yes)
+		(on_board yes)
+		(dnp no)
+		(fields_autoplaced yes)
+		(property "Reference" "TP2"
+			(at 134.62 20.3199 90)
+			(effects
+				(font
+					(size 1.27 1.27)
+				)
+				(justify left)
+			)
+		)
+		(property "Value" "TestPoint"
+			(at 134.62 22.8599 90)
+			(effects
+				(font
+					(size 1.27 1.27)
+				)
+				(justify left)
+			)
+		)
+		(property "Footprint" "TestPoint:TestPoint_Plated_Hole_D2.0mm"
+			(at 129.54 26.67 0)
+			(effects
+				(font
+					(size 1.27 1.27)
+				)
+				(hide yes)
+			)
+		)
+		(property "Datasheet" "~"
+			(at 129.54 26.67 0)
+			(effects
+				(font
+					(size 1.27 1.27)
+				)
+				(hide yes)
+			)
+		)
+		(property "Description" "test point"
+			(at 129.54 21.59 0)
+			(effects
+				(font
+					(size 1.27 1.27)
+				)
+				(hide yes)
+			)
+		)
+		(pin "1"
+		)
+		(instances
+			(project "TwinklePad"
+				(path "/16706bee-9459-4bee-94a4-70f692e45dc3"
+					(reference "TP2")
+					(unit 1)
+				)
+			)
+		)
+	)
+	(symbol
 		(lib_id "Switch:SW_Push")
 		(at 224.79 104.14 0)
@@
 	(symbol
 		(lib_id "power:GND")
-		(at 132.08 29.21 0)
+		(at 129.54 31.75 0)
 		(unit 1)
 		(exclude_from_sim no)
@@
 		(dnp no)
 		(property "Reference" "#PWR01"
-			(at 132.08 35.56 0)
+			(at 129.54 38.1 0)
 			(effects
 				(font
@@
 		)
 		(property "Value" "GND"
-			(at 132.08 34.29 0)
+			(at 129.54 36.83 0)
 			(effects
 				(font
@@
 		)
 		(property "Footprint" ""
-			(at 132.08 29.21 0)
+			(at 129.54 31.75 0)
 			(effects
 				(font
@@
 		)
 		(property "Datasheet" ""
-			(at 132.08 29.21 0)
+			(at 129.54 31.75 0)
 			(effects
 				(font
@@
 		)
 		(property "Description" "Power symbol creates a global label with name \"GND\" , ground"
-			(at 132.08 29.21 0)
+			(at 129.54 31.75 0)
 			(effects
 				(font
@@
 	(symbol
 		(lib_id "power:VCC")
-		(at 132.08 16.51 90)
+		(at 129.54 16.51 90)
 		(unit 1)
 		(exclude_from_sim no)
@@
 		(fields_autoplaced yes)
 		(property "Reference" "#PWR02"
-			(at 135.89 16.51 0)
+			(at 133.35 16.51 0)
 			(effects
 				(font
@@
 		)
 		(property "Value" "VCC"
-			(at 128.27 16.5099 90)
+			(at 125.73 16.5099 90)
 			(effects
 				(font
@@
 		)
 		(property "Footprint" ""
-			(at 132.08 16.51 0)
+			(at 129.54 16.51 0)
 			(effects
 				(font
@@
 		)
 		(property "Datasheet" ""
-			(at 132.08 16.51 0)
+			(at 129.54 16.51 0)
 			(effects
 				(font
@@
 		)
 		(property "Description" "Power symbol creates a global label with name \"VCC\""
-			(at 132.08 16.51 0)
+			(at 129.54 16.51 0)
 			(effects
 				(font
