File: TwinklePad.kicad_pcb (KiCad board)
At the start: 2 copper layers, 86 x 124 mm, 63 parts, among them J1 Conn_01x04_Pin, J2 Conn_01x02, J4 PRT-12639, Q1 S8050, SW1 SW_Push, SW10 SW_Push, SW11 SW_Push, SW12 SW_Push, SW13 SW_Push, SW14 SW_Push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

Commit message: Finished pcb, schematic and positioning - more or less
Parts:
- removed J2: Conn_01x02, Connector_PinHeader_2.54mm:PinHeader_1x02_P2.54mm_Vertical
- added BUZ+: TestPoint, TestPoint:TestPoint_Plated_Hole_D2.0mm, F.Cu at (126.5, 54.0)
- added BUZ-: TestPoint, TestPoint:TestPoint_Plated_Hole_D2.0mm, F.Cu at (130.5, 54.0)
- added REF**: MountingHole_3.2mm_M3, MountingHole:MountingHole_3.2mm_M3, F.Cu at (128.8, 46.0)
- J4: moved to F.Cu
- Q1: footprint Package_TO_SOT_THT:TO-92_Inline -> Package_TO_SOT_THT:TO-92_Inline_Horizontal1; moved to B.Cu
- moved Q1 4.34 mm to (131.5, 57.0), turned to 180 degrees
- moved JP1 3.76 mm to (122.6, 30.2)
- moved REC_B1 2.21 mm to (179.7, 66.5)
- moved J1 1.80 mm to (123.7, 58.1)
- moved REC_A1 1.41 mm to (105.7, 61.5)
- moved J4 1.08 mm to (127.0, 34.4)
- moved S1 0.83 mm to (118.2, 38.5)
Routing:
- net VCC: track 539.3 -> 526.6 mm, vias 28 -> 25
- net +3.3V: track 107.7 -> 101.1 mm, vias 5 -> 4
- net RX: track 63.4 -> 57.3 mm, vias 1 -> 0
- net GND: track 16.9 -> 11.7 mm
- net Net-(JP1-A): track 4.47 -> 8.44 mm, vias 0 -> 1
- net OLED_SCL: track 33.9 -> 30.1 mm, vias 3 -> 1
- net REC_SW_B2: track 12.4 -> 15.8 mm, vias 0 -> 1
- net ROW 3: track 185.2 -> 188.2 mm
- net REC_A1: track 67.7 -> 70.5 mm
- net REC_B1: track 72.6 -> 75.3 mm
- net REC_B2: track 69.5 -> 67.1 mm
- net Buzzer+: track 16.9 -> 19.1 mm
- net REC_A2: track 58.8 -> 60.8 mm
- net ROW 2: track 160.1 -> 162.1 mm
- net COL 0: track 154.4 -> 156.1 mm
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Other:
- board size 86 x 124 mm -> 84 x 124 mm

Commit message: Did some minor changes
Parts:
- D17, D18, D19, D20, D21, D22, D23, D24, D25, D26, D27, D28, D29, D30, D31, D32, D33, D34: moved to B.Cu
Routing:
- net GND: track 11.7 -> 14.1 mm, vias 6 -> 8
- net REC_B2: track 67.1 -> 66.3 mm
